File: Schematics/Optimized/Fiu/pg_13.kicad_sch (KiCad schematic)
At the start: 1 part, among them U29 XREG64

Commit message: FIU: integrate entire rotor
Tested: passed run_udiag on r2000
Tested: passed boot_env (fiu-5d8246), until PRETTY_PRINTER exception
Parts:
- added U702: XREG64, symbol r1000:XREG64
Connections:
- new net VAR.SCLK: U702.1 (CLK)
- new net VAR_VI.OE~: U702.3 (OE)
- new net VI.D0: U702.7 (Q0)
- new net VI.D1: U702.9 (Q1)
- new net VI.D10: U702.27 (Q10)
- new net VI.D11: U702.29 (Q11)
- new net VI.D12: U702.31 (Q12)
- new net VI.D13: U702.33 (Q13)
- new net VI.D14: U702.35 (Q14)
- new net VI.D15: U702.37 (Q15)
- new net VI.D16: U702.39 (Q16)
- new net VI.D17: U702.41 (Q17)
- new net VI.D18: U702.43 (Q18)
- new net VI.D19: U702.45 (Q19)
- new net VI.D2: U702.11 (Q2)
- new net VI.D20: U702.47 (Q20)
- new net VI.D21: U702.49 (Q21)
- new net VI.D22: U702.51 (Q22)
- new net VI.D23: U702.53 (Q23)
- new net VI.D24: U702.55 (Q24)
- new net VI.D25: U702.57 (Q25)
- new net VI.D26: U702.59 (Q26)
- new net VI.D27: U702.61 (Q27)
- new net VI.D28: U702.63 (Q28)
- new net VI.D29: U702.65 (Q29)
- new net VI.D3: U702.13 (Q3)
- new net VI.D30: U702.67 (Q30)
- new net VI.D31: U702.69 (Q31)
- new net VI.D32: U702.71 (Q32)
- new net VI.D33: U702.73 (Q33)
- new net VI.D34: U702.75 (Q34)
- new net VI.D35: U702.77 (Q35)
- new net VI.D36: U702.79 (Q36)
- new net VI.D37: U702.81 (Q37)
- new net VI.D38: U702.83 (Q38)
- new net VI.D39: U702.85 (Q39)
- new net VI.D4: U702.15 (Q4)
- new net VI.D40: U702.87 (Q40)
- new net VI.D41: U702.89 (Q41)
- new net VI.D42: U702.91 (Q42)
- new net VI.D43: U702.93 (Q43)
- new net VI.D44: U702.95 (Q44)
- new net VI.D45: U702.97 (Q45)
- new net VI.D46: U702.99 (Q46)
- new net VI.D47: U702.101 (Q47)
- new net VI.D48: U702.103 (Q48)
- new net VI.D49: U702.105 (Q49)
- new net VI.D5: U702.17 (Q5)
- new net VI.D50: U702.107 (Q50)
- new net VI.D51: U702.109 (Q51)
- new net VI.D52: U702.111 (Q52)
- new net VI.D53: U702.113 (Q53)
- new net VI.D54: U702.115 (Q54)
- new net VI.D55: U702.117 (Q55)
- new net VI.D56: U702.119 (Q56)
- new net VI.D57: U702.121 (Q57)
- new net VI.D58: U702.123 (Q58)
- new net VI.D59: U702.125 (Q59)
- new net VI.D6: U702.19 (Q6)
- new net VI.D60: U702.127 (Q60)
- new net VI.D61: U702.129 (Q61)
- new net VI.D62: U702.131 (Q62)
- new net VI.D63: U702.133 (Q63)
- new net VI.D7: U702.21 (Q7)
- new net VI.D8: U702.23 (Q8)
- new net VI.D9: U702.25 (Q9)
- new net VO.D0: U702.6 (D0)
- new net VO.D1: U702.8 (D1)
- new net VO.D10: U702.26 (D10)
- new net VO.D11: U702.28 (D11)
- new net VO.D12: U702.30 (D12)
- new net VO.D13: U702.32 (D13)
- new net VO.D14: U702.34 (D14)
- new net VO.D15: U702.36 (D15)
- new net VO.D16: U702.38 (D16)
- new net VO.D17: U702.40 (D17)
- new net VO.D18: U702.42 (D18)
- new net VO.D19: U702.44 (D19)
- new net VO.D2: U702.10 (D2)
- new net VO.D20: U702.46 (D20)
- new net VO.D21: U702.48 (D21)
- new net VO.D22: U702.50 (D22)
- new net VO.D23: U702.52 (D23)
- new net VO.D24: U702.54 (D24)
- new net VO.D25: U702.56 (D25)
- new net VO.D26: U702.58 (D26)
- new net VO.D27: U702.60 (D27)
- new net VO.D28: U702.62 (D28)
- new net VO.D29: U702.64 (D29)
- new net VO.D3: U702.12 (D3)
- new net VO.D30: U702.66 (D30)
- new net VO.D31: U702.68 (D31)
- new net VO.D32: U702.70 (D32)
- new net VO.D33: U702.72 (D33)
- new net VO.D34: U702.74 (D34)
- new net VO.D35: U702.76 (D35)
- new net VO.D36: U702.78 (D36)
- new net VO.D37: U702.80 (D37)
- new net VO.D38: U702.82 (D38)
- new net VO.D39: U702.84 (D39)
- new net VO.D4: U702.14 (D4)
- new net VO.D40: U702.86 (D40)
- new net VO.D41: U702.88 (D41)
- new net VO.D42: U702.90 (D42)
- new net VO.D43: U702.92 (D43)
- new net VO.D44: U702.94 (D44)
- new net VO.D45: U702.96 (D45)
- new net VO.D46: U702.98 (D46)
- new net VO.D47: U702.100 (D47)
- new net VO.D48: U702.102 (D48)
- new net VO.D49: U702.104 (D49)
- new net VO.D5: U702.16 (D5)
- new net VO.D50: U702.106 (D50)
- new net VO.D51: U702.108 (D51)
- new net VO.D52: U702.110 (D52)
- new net VO.D53: U702.112 (D53)
- new net VO.D54: U702.114 (D54)
- new net VO.D55: U702.116 (D55)
- new net VO.D56: U702.118 (D56)
- new net VO.D57: U702.120 (D57)
- new net VO.D58: U702.122 (D58)
- new net VO.D59: U702.124 (D59)
- new net VO.D6: U702.18 (D6)
- new net VO.D60: U702.126 (D60)
- new net VO.D61: U702.128 (D61)
- new net VO.D62: U702.130 (D62)
- new net VO.D63: U702.132 (D63)
- new net VO.D7: U702.20 (D7)
- new net VO.D8: U702.22 (D8)
- new net VO.D9: U702.24 (D9)
- no-connect marks 1 -> 2
Other:
- moved on the sheet: U29
