File: Schematics/Optimized/Val/pg_17.kicad_sch (KiCad schematic)
At the start: 2 parts, among them U42 XMUX32, U43 XMUX32

Commit message: Polish
Tested: passed expmon_test_{typ,val} (-busmux)
Tested: passed run_udiag on r2000
Other:
- moved on the sheet: U42, U43
