File: Schematics/Optimized/Seq/pg_43.kicad_sch (KiCad schematic)
At the start: 16 parts, among them U114 XPAR32, U4407 F240, U4408 F374, U4409 F521, U4410 F51, U4411 F37, U81 XPAR18

Commit message: Replace BUZZ_OFF~ with Q1~
Connections:
- net Q.BUZZ_OFF~ renamed Q1~
Changed lines of the file:
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@@
     )
   )
-  (global_label "Q.BUZZ_OFF~" (shape input) (at 378.46 243.84 180) (fields_autoplaced)
+  (global_label "Q1~" (shape input) (at 378.46 243.84 180) (fields_autoplaced)
     (effects (font (size 2.54 2.54)) (justify right))
-    (property "Intersheetrefs" "${INTERSHEET_REFS}" (at 348.9597 243.6813 0)
+    (property "Intersheetrefs" "${INTERSHEET_REFS}" (at 365.5647 243.84 0)
       (effects (font (size 1.905 1.905)) (justify right))
     )

Commit message: SEQ condensation
Tested: passed run_udiag
Tested: passed expmon_test_seq --quick
Tested: 16.7s (&c) boot_env
Changed lines of the file:
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@@
-    (stroke (width 0) (type default))
-  )
-  (bus (pts (xy 396.24 142.24) (xy 396.24 147.32))
     (stroke (width 0) (type default))
   )
@@
     (stroke (width 0) (type default))
   )
+  (wire (pts (xy 490.22 114.3) (xy 490.22 116.84))
+    (stroke (width 0) (type default))
+  )
   (wire (pts (xy 495.3 142.24) (xy 530.86 142.24))
     (stroke (width 0) (type default))
   )
-  (wire (pts (xy 482.6 114.3) (xy 497.84 114.3))
+  (wire (pts (xy 482.6 114.3) (xy 490.22 114.3))
     (stroke (width 0) (type default))
   )
@@
     (stroke (width 0) (type default))
   )
-  (wire (pts (xy 464.82 88.9) (xy 474.98 88.9))
+  (wire (pts (xy 469.9 114.3) (xy 474.98 114.3))
     (stroke (width 0) (type default))
   )
@@
     (stroke (width 0) (type default))
   )
-  (wire (pts (xy 474.98 88.9) (xy 474.98 116.84))
+  (wire (pts (xy 474.98 114.3) (xy 474.98 116.84))
     (stroke (width 0) (type default))
   )
@@
     )
   )
-  (global_label "~LOCAL.CLK~" (shape input) (at 464.82 88.9 180) (fields_autoplaced)
+  (global_label "~LOCAL.CLK~" (shape input) (at 469.9 114.3 180) (fields_autoplaced)
     (effects (font (size 2.54 2.54)) (justify right))
-    (property "Intersheetrefs" "${INTERSHEET_REFS}" (at 436.5292 88.7413 0)
+    (property "Intersheetrefs" "${INTERSHEET_REFS}" (at 441.6092 114.1413 0)
       (effects (font (size 1.905 1.905)) (justify right))
     )
@@
     )
   )
-  (symbol (lib_id "r1000:PD") (at 497.84 114.3 0) (unit 1)
+  (symbol (lib_id "r1000:PD") (at 490.22 116.84 0) (unit 1)
     (in_bom no) (on_board yes) (dnp no)
-    (property "Reference" "#PWR0143" (at 497.84 114.3 0)
-      (effects (font (size 1.27 1.27)) hide)
-    )
-    (property "Value" "PD" (at 497.84 114.3 0)
-      (effects (font (size 1.27 1.27)) hide)
-    )
-    (property "Footprint" "" (at 497.84 114.3 0)
-      (effects (font (size 1.27 1.27)) hide)
-    )
-    (property "Datasheet" "" (at 497.84 114.3 0)
-      (effects (font (size 1.27 1.27)) hide)
-    )
+    (property "Reference" "#PWR0143" (at 490.22 116.84 0)
+      (effects (font (size 1.27 1.27)) hide)
+    )
+    (property "Value" "PD" (at 490.22 116.84 0)
+      (effects (font (size 1.27 1.27)) hide)
+    )
+    (property "Footprint" "" (at 490.22 116.84 0)
+      (effects (font (size 1.27 1.27)) hide)
+    )
+    (property "Datasheet" "" (at 490.22 116.84 0)
+      (effects (font (size 1.27 1.27)) hide)
+    )
