File: Schematics/Optimized/Seq/pg_36.kicad_sch (KiCad schematic)
At the start: 80 parts, among them U90 XBUF32, U91 XBUF20, U92 XBUF16, U93 XBUF20

Commit message: SEQ condensation
Tested: passed run_udiag
Tested: passed expmon_test_seq --quick
Tested: 16.7s (&c) boot_env
Parts:
- removed U91, U93: XBUF20, symbol r1000:XBUF20
- removed U92: XBUF16, symbol r1000:XBUF16
- added GB264: GB, symbol r1000:GB
- added U1602: XBUF3, symbol r1000:XBUF3
- added U1603: XMUX32, symbol r1000:XMUX32
- added U1617: XBUF20, symbol r1000:XBUF20
- added U3818: F04, symbol r1000:F04
- added U3819: F00, symbol r1000:F00
- added U3821: F51, symbol r1000:F51
- added U3823, U3824: F37, symbol r1000:F37
Connections:
- net ADR.OFFS~37: now also U1603.47 (B5)
- net ADR.OFFS~38: now also U1603.49 (B6)
- net ADR.OFFS~39: now also U1603.51 (B7)
- net ADR.OFFS~40: now also U1603.53 (B8)
- net ADR.OFFS~41: now also U1603.55 (B9)
- net ADR.OFFS~42: now also U1603.57 (B10)
- net ADR.OFFS~43: now also U1603.59 (B11)
- net ADR.OFFS~44: now also U1603.61 (B12)
- net ADR.OFFS~45: now also U1603.63 (B13)
- net ADR.OFFS~46: now also U1603.65 (B14)
- net ADR.OFFS~47: now also U1603.67 (B15)
- net ADR.OFFS~48: now also U1603.69 (B16)
- net ADR.OFFS~49: now also U1603.71 (B17)
- net ADR.OFFS~50: now also U1603.73 (B18)
- net ADR.OFFS~51: now also U1603.75 (B19)
- net ADR.OFFS~52: now also U1603.77 (B20)
- net ADR.OFFS~53: now also U1603.79 (B21)
- net ADR.OFFS~54: now also U1603.81 (B22)
- net ADR.OFFS~55: now also U1603.83 (B23)
- net ADR.OFFS~56: now also U1603.85 (B24)
- net ADR.SPACE~0: now also U1602.3 (I0)
- net ADR.SPACE~1: now also U1602.5 (I1)
- net ADR.SPACE~2: now also U1602.7 (I2)
- net BRANCH.IND~57: now also U1603.30 (A25), U1603.87 (B25)
- net BRANCH.IND~58: now also U1603.31 (A26), U1603.89 (B26)
- net BRANCH.IND~59: now also U1603.32 (A27), U1603.91 (B27)
- net NAME_SPACE.OE~: now also U1602.2 (OE), U1603.8 (OE), U3824.3 (Q)
- net OFFSET.OE~: now also U3823.3 (Q)
- net PD: now also U1602.1 (INV), U1603.2 (INV), U1603.6 (E), U1617.1 (INV), U1617.2 (OE)
- net Q.ADR.OFFS0: now also U1603.38 (Y0)
- net Q.ADR.OFFS1: now also U1603.40 (Y1)
- net Q.ADR.OFFS10: now also U1603.58 (Y10)
- net Q.ADR.OFFS11: now also U1603.60 (Y11)
- net Q.ADR.OFFS12: now also U1603.62 (Y12)
- net Q.ADR.OFFS13: now also U1603.64 (Y13)
- net Q.ADR.OFFS14: now also U1603.66 (Y14)
- net Q.ADR.OFFS15: now also U1603.68 (Y15)
- net Q.ADR.OFFS16: now also U1603.70 (Y16)
- net Q.ADR.OFFS17: now also U1603.72 (Y17)
- net Q.ADR.OFFS18: now also U1603.74 (Y18)
- net Q.ADR.OFFS19: now also U1603.76 (Y19)
- net Q.ADR.OFFS2: now also U1603.42 (Y2)
- net Q.ADR.OFFS20: now also U1603.78 (Y20)
- net Q.ADR.OFFS21: now also U1603.80 (Y21)
- net Q.ADR.OFFS22: now also U1603.82 (Y22)
- net Q.ADR.OFFS23: now also U1603.84 (Y23)
- net Q.ADR.OFFS24: now also U1603.86 (Y24)
- net Q.ADR.OFFS25: now also U1603.88 (Y25)
- net Q.ADR.OFFS26: now also U1603.90 (Y26)
- net Q.ADR.OFFS27: now also U1603.92 (Y27)
- net Q.ADR.OFFS28: now also U1603.94 (Y28)
- net Q.ADR.OFFS29: now also U1603.96 (Y29)
- net Q.ADR.OFFS3: now also U1603.44 (Y3)
- net Q.ADR.OFFS30: now also U1603.98 (Y30)
- net Q.ADR.OFFS31: now also U1603.100 (Y31)
- net Q.ADR.OFFS4: now also U1603.46 (Y4)
- net Q.ADR.OFFS5: now also U1603.48 (Y5)
- net Q.ADR.OFFS6: now also U1603.50 (Y6)
- net Q.ADR.OFFS7: now also U1603.52 (Y7)
- net Q.ADR.OFFS8: now also U1603.54 (Y8)
- net Q.ADR.OFFS9: now also U1603.56 (Y9)
- net Q.ADR.SPACE0: now also U1602.4 (Y0)
- net Q.ADR.SPACE1: now also U1602.6 (Y1)
- net Q.ADR.SPACE2: now also U1602.8 (Y2)
- net RESOLVE_OFFS37: now also U1617.3 (I0)
- net RESOLVE_OFFS38: now also U1617.5 (I1)
- net RESOLVE_OFFS39: now also U1617.7 (I2)
- net RESOLVE_OFFS40: now also U1617.9 (I3)
- net RESOLVE_OFFS41: now also U1617.11 (I4)
- net RESOLVE_OFFS42: now also U1617.13 (I5)
- net RESOLVE_OFFS43: now also U1617.15 (I6)
- net RESOLVE_OFFS44: now also U1617.17 (I7)
- net RESOLVE_OFFS45: now also U1617.19 (I8)
- net RESOLVE_OFFS46: now also U1617.21 (I9)
- net RESOLVE_OFFS47: now also U1617.23 (I10)
- net RESOLVE_OFFS48: now also U1617.25 (I11)
- net RESOLVE_OFFS49: now also U1617.27 (I12)
- net RESOLVE_OFFS50: now also U1617.29 (I13)
- net RESOLVE_OFFS51: now also U1617.31 (I14)
- net RESOLVE_OFFS52: now also U1617.33 (I15)
- net RESOLVE_OFFS53: now also U1617.35 (I16)
- net RESOLVE_OFFS54: now also U1617.37 (I17)
- net RESOLVE_OFFS55: now also U1617.39 (I18)
- net RESOLVE_OFFS56: now also U1617.41 (I19)
- new net: U3818.2 (Q), U3821.2 (A2)
- new net: U3821.7 (Q), U3823.1 (D0)
- new net: U1603.13 (A8), U1617.10 (Y3)
- new net: U1603.14 (A9), U1617.12 (Y4)
- new net: U1603.15 (A10), U1617.14 (Y5)
- new net: U1603.16 (A11), U1617.16 (Y6)
- new net: U1603.17 (A12), U1617.18 (Y7)
- new net: U1603.18 (A13), U1617.20 (Y8)
- new net: U1603.19 (A14), U1617.22 (Y9)
- new net: U1603.20 (A15), U1617.24 (Y10)
- new net: U1603.21 (A16), U1617.26 (Y11)
- new net: U1603.22 (A17), U1617.28 (Y12)
- new net: U1603.23 (A18), U1617.30 (Y13)
- new net: U1603.24 (A19), U1617.32 (Y14)
- new net: U1603.25 (A20), U1617.34 (Y15)
- new net: U1603.26 (A21), U1617.36 (Y16)
- new net: U1603.27 (A22), U1617.38 (Y17)
- new net: U1603.10 (A5), U1617.4 (Y0)
- new net: U1603.28 (A23), U1617.40 (Y18)
- new net: U1603.29 (A24), U1617.42 (Y19)
- new net: U1603.11 (A6), U1617.6 (Y1)
- new net: U1603.12 (A7), U1617.8 (Y2)
- new net: U3819.3 (Q), U3824.1 (D0)
- new net ADR_OFF.DIAG~: U3823.2 (D1), U3824.2 (D1)
- new net ADR_ON.DIAG~: U3819.2 (D1), U3821.3 (A3), U3821.6 (B3)
- new net Q.SEQ_A.EN~: GB264.1, U3819.1 (D0), U3821.5 (B2)
- new net RESOLVE_DRIVE~: U1603.4 (S), U3818.1 (D0)
- no-connect marks 3 -> 20
Other:
- moved on the sheet: GB101, GB102, GB104, GB105, GB14, GB145, GB146, GB147, GB15, GB153, GB154, GB155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

Commit message: Merge SEQ changes
Tested: passed run_udiag
Parts:
- removed GB145, GB146, GB147, GB153, GB154, GB155, GB157, GB158, GB161: GB, symbol r1000:GB

Commit message: Condensation of SEQ, TYP & VAL conditions
Parts:
- removed U1603: XMUX32, symbol r1000:XMUX32
- removed U1617: XBUF20, symbol r1000:XBUF20
- removed U3818: F04, symbol r1000:F04
- removed U3821: F51, symbol r1000:F51
- removed U3823: F37, symbol r1000:F37
- added GB145, GB146, GB147, GB153, GB154, GB155, GB157, GB158, GB161: GB, symbol r1000:GB
- added U1001: XMUX32, symbol r1000:XMUX32
- added U1715: F04, symbol r1000:F04
- added U1716: F00, symbol r1000:F00
- added U3801: XPAR32, symbol r1000:XPAR32
- added U3829: F374, symbol r1000:F374
- added U906: XSEQOFS, symbol r1000:XSEQOFS
- added U907: XREG9, symbol r1000:XREG9
Connections:
- net ADR_OFF.DIAG~: now also U3824.1 (D0); no longer U3824.2 (D1)
- net BRANCH.IND~57: now also U906.92 (BRNC0)
- net BRANCH.IND~58: now also U906.93 (BRNC1)
- net BRANCH.IND~59: now also U906.94 (BRNC2)
- net NAME_SPACE.OE~: now also U1715.1 (D0), U906.2 (OE)
- net PD: now also U1001.37 (B0), U1001.39 (B1), U1001.41 (B2), U1001.43 (B3), U1001.45 (B4), U1001.47 (B5), U1001.49 (B6), U1001.51 (B7), U1001.6 (E), U1001.8 (OE), U3829.1 (OE), U907.2 (INV); no longer U90.1 (INV)
- net Q.ADR.OFFS0: now also U906.4 (ADR0)
- net Q.ADR.OFFS1: now also U906.5 (ADR1)
- net Q.ADR.OFFS10: now also U906.23 (ADR10)
- net Q.ADR.OFFS11: now also U906.25 (ADR11)
- net Q.ADR.OFFS12: now also U906.27 (ADR12)
- net Q.ADR.OFFS13: now also U906.29 (ADR13)
- net Q.ADR.OFFS14: now also U906.31 (ADR14)
- net Q.ADR.OFFS15: now also U906.33 (ADR15)
- net Q.ADR.OFFS16: now also U906.35 (ADR16)
- net Q.ADR.OFFS17: now also U906.37 (ADR17)
- net Q.ADR.OFFS18: now also U906.39 (ADR18)
- net Q.ADR.OFFS19: now also U906.41 (ADR19)
- net Q.ADR.OFFS2: now also U906.7 (ADR2)
- net Q.ADR.OFFS20: now also U906.43 (ADR20)
- net Q.ADR.OFFS21: now also U906.45 (ADR21)
- net Q.ADR.OFFS22: now also U906.46 (ADR22)
- net Q.ADR.OFFS23: now also U906.48 (ADR23)
- net Q.ADR.OFFS24: now also U906.50 (ADR24)
- net Q.ADR.OFFS25: now also U906.52 (ADR25)
- net Q.ADR.OFFS26: now also U906.54 (ADR26)
- net Q.ADR.OFFS27: now also U906.56 (ADR27)
- net Q.ADR.OFFS28: now also U906.58 (ADR28)
- net Q.ADR.OFFS29: now also U906.60 (ADR29)
- net Q.ADR.OFFS3: now also U906.9 (ADR3)
- net Q.ADR.OFFS30: now also U906.62 (ADR30)
- net Q.ADR.OFFS31: now also U906.64 (ADR31)
- net Q.ADR.OFFS4: now also U906.11 (ADR4)
- net Q.ADR.OFFS5: now also U906.13 (ADR5)
- net Q.ADR.OFFS6: now also U906.15 (ADR6)
- net Q.ADR.OFFS7: now also U906.17 (ADR7)
- net Q.ADR.OFFS8: now also U906.19 (ADR8)
- net Q.ADR.OFFS9: now also U906.21 (ADR9)
- net RESOLVE_DRIVE~: now also U906.1 (RESDR)
- net RESOLVE_OFFS37: now also U906.6 (RES0)
- net RESOLVE_OFFS38: now also U906.8 (RES1)
- net RESOLVE_OFFS39: now also U906.10 (RES2)
- net RESOLVE_OFFS40: now also U906.12 (RES3)
- net RESOLVE_OFFS41: now also U906.14 (RES4)
- net RESOLVE_OFFS42: now also U906.16 (RES5)
- net RESOLVE_OFFS43: now also U906.18 (RES6)
- net RESOLVE_OFFS44: now also U906.20 (RES7)
- net RESOLVE_OFFS45: now also U906.22 (RES8)
- net RESOLVE_OFFS46: now also U906.24 (RES9)
- net RESOLVE_OFFS47: now also U906.26 (RES10)
- net RESOLVE_OFFS48: now also U906.28 (RES11)
- net RESOLVE_OFFS49: now also U906.30 (RES12)
- net RESOLVE_OFFS50: now also U906.32 (RES13)
- net RESOLVE_OFFS51: now also U906.34 (RES14)
- net RESOLVE_OFFS52: now also U906.36 (RES15)
- net RESOLVE_OFFS53: now also U906.38 (RES16)
- net RESOLVE_OFFS54: now also U906.40 (RES17)
- net RESOLVE_OFFS55: now also U906.42 (RES18)
- net RESOLVE_OFFS56: now also U906.44 (RES19)
- net at U3819.3 (Q): now also U3824.2 (D1); no longer U3824.1 (D0)
- net ADR.NAME~0 renamed ADR.NAME0
- net ADR.NAME0: now also U1001.38 (Y0), U3801.2 (I0)
- net ADR.NAME~1 renamed ADR.NAME1
- net ADR.NAME1: now also U1001.40 (Y1), U3801.4 (I1)
- net ADR.NAME~10 renamed ADR.NAME10
- net ADR.NAME10: now also U1001.58 (Y10), U3801.17 (I10)
- net ADR.NAME~11 renamed ADR.NAME11
- net ADR.NAME11: now also U1001.60 (Y11), U3801.18 (I11)
- net ADR.NAME~12 renamed ADR.NAME12
- net ADR.NAME12: now also U1001.62 (Y12), U3801.19 (I12)
- net ADR.NAME~13 renamed ADR.NAME13
- net ADR.NAME13: now also U1001.64 (Y13), U3801.20 (I13)
- net ADR.NAME~14 renamed ADR.NAME14
- net ADR.NAME14: now also U1001.66 (Y14), U3801.21 (I14)
- net ADR.NAME~15 renamed ADR.NAME15
- net ADR.NAME15: now also U1001.68 (Y15), U3801.22 (I15)
- net ADR.NAME~16 renamed ADR.NAME16
- net ADR.NAME16: now also U1001.70 (Y16), U3801.23 (I16)
- net ADR.NAME~17 renamed ADR.NAME17
- net ADR.NAME17: now also U1001.72 (Y17), U3801.24 (I17)
- net ADR.NAME~18 renamed ADR.NAME18
- net ADR.NAME18: now also U1001.74 (Y18), U3801.25 (I18)
- net ADR.NAME~19 renamed ADR.NAME19
- net ADR.NAME19: now also U1001.76 (Y19), U3801.26 (I19)
- net ADR.NAME~2 renamed ADR.NAME2
- net ADR.NAME2: now also U1001.42 (Y2), U3801.6 (I2)
- net ADR.NAME~20 renamed ADR.NAME20
- net ADR.NAME20: now also U1001.78 (Y20), U3801.27 (I20)
- net ADR.NAME~21 renamed ADR.NAME21
- net ADR.NAME21: now also U1001.80 (Y21), U3801.28 (I21)
- net ADR.NAME~22 renamed ADR.NAME22
- net ADR.NAME22: now also U1001.82 (Y22), U3801.29 (I22)
- net ADR.NAME~23 renamed ADR.NAME23
- net ADR.NAME23: now also U1001.84 (Y23), U3801.30 (I23)
- net ADR.NAME~24 renamed ADR.NAME24
- net ADR.NAME24: now also U1001.86 (Y24), U3801.31 (I24)
- net ADR.NAME~25 renamed ADR.NAME25
- net ADR.NAME25: now also U1001.88 (Y25), U3801.32 (I25)
- net ADR.NAME~26 renamed ADR.NAME26
- net ADR.NAME26: now also U1001.90 (Y26), U3801.33 (I26)
- net ADR.NAME~27 renamed ADR.NAME27
- net ADR.NAME27: now also U1001.92 (Y27), U3801.34 (I27)
- net ADR.NAME~28 renamed ADR.NAME28
- net ADR.NAME28: now also U1001.94 (Y28), U3801.35 (I28)
- net ADR.NAME~29 renamed ADR.NAME29
- net ADR.NAME29: now also U1001.96 (Y29), U3801.36 (I29)
- net ADR.NAME~3 renamed ADR.NAME3
- net ADR.NAME3: now also U1001.44 (Y3), U3801.8 (I3)
- net ADR.NAME~30 renamed ADR.NAME30
- net ADR.NAME30: now also U1001.98 (Y30), U3801.37 (I30)
- net ADR.NAME~31 renamed ADR.NAME31
- net ADR.NAME31: now also U1001.100 (Y31), U3801.38 (I31)
- net ADR.NAME~4 renamed ADR.NAME4
- net ADR.NAME4: now also U1001.46 (Y4), U3801.10 (I4)
- net ADR.NAME~5 renamed ADR.NAME5
- net ADR.NAME5: now also U1001.48 (Y5), U3801.11 (I5)
- net ADR.NAME~6 renamed ADR.NAME6
- net ADR.NAME6: now also U1001.50 (Y6), U3801.12 (I6)
- net ADR.NAME~7 renamed ADR.NAME7
- net ADR.NAME7: now also U1001.52 (Y7), U3801.13 (I7)
- net ADR.NAME~8 renamed ADR.NAME8
- net ADR.NAME8: now also U1001.54 (Y8), U3801.14 (I8)
- net ADR.NAME~9 renamed ADR.NAME9
- net ADR.NAME9: now also U1001.56 (Y9), U3801.15 (I9)
- new net: U1716.3 (Q), U907.3 (OE)
- new net: U1716.2 (D1), U3829.2 (Q0)
- new net: U1715.2 (Q), U3829.3 (D0)
- new net ADR.SPACE_PEV: U907.6 (D0)
- new net ADR_IS_CODE: U1001.4 (S), U906.3 (ADRIC)
- new net BIT_PEV: U906.72 (PAR3), U907.22 (D8)
- new net CODE.OFFS45: U906.47 (CODE0)
- new net CODE.OFFS46: U906.49 (CODE1)
- new net CODE.OFFS47: U906.51 (CODE2)
- new net CODE.OFFS48: U906.53 (CODE3)
- new net CODE.OFFS49: U906.55 (CODE4)
- new net CODE.OFFS50: U906.57 (CODE5)
- new net CODE.OFFS51: U906.59 (CODE6)
- new net CODE.OFFS52: U906.61 (CODE7)
- new net CODE.OFFS53: U906.63 (CODE8)
- new net CODE.OFFS54: U906.65 (CODE9)
- new net CODE.OFFS55: U906.66 (CODE10)
- new net CODE.OFFS56: U906.68 (CODE11)
- new net CODE.SEGN10: U1001.57 (B10)
- new net CODE.SEGN11: U1001.59 (B11)
- new net CODE.SEGN12: U1001.61 (B12)
- new net CODE.SEGN13: U1001.63 (B13)
- new net CODE.SEGN14: U1001.65 (B14)
- new net CODE.SEGN15: U1001.67 (B15)
- new net CODE.SEGN16: U1001.69 (B16)
- new net CODE.SEGN17: U1001.71 (B17)
- new net CODE.SEGN18: U1001.73 (B18)
- new net CODE.SEGN19: U1001.75 (B19)
- new net CODE.SEGN20: U1001.77 (B20)
- new net CODE.SEGN21: U1001.79 (B21)
- new net CODE.SEGN22: U1001.81 (B22)
- new net CODE.SEGN23: U1001.83 (B23)
- new net CODE.SEGN24: U1001.85 (B24)
- new net CODE.SEGN25: U1001.87 (B25)
- new net CODE.SEGN26: U1001.89 (B26)
- new net CODE.SEGN27: U1001.91 (B27)
- new net CODE.SEGN28: U1001.93 (B28)
- new net CODE.SEGN29: U1001.95 (B29)
- new net CODE.SEGN30: U1001.97 (B30)
- new net CODE.SEGN31: U1001.99 (B31)
- new net CODE.SEGN8: U1001.53 (B8)
- new net CODE.SEGN9: U1001.55 (B9)
- new net NAME_BUS0: U1001.1 (A0)
- new net NAME_BUS1: U1001.3 (A1)
- new net NAME_BUS10: U1001.15 (A10)
- new net NAME_BUS11: U1001.16 (A11)
- new net NAME_BUS12: U1001.17 (A12)
- new net NAME_BUS13: U1001.18 (A13)
- new net NAME_BUS14: U1001.19 (A14)
- new net NAME_BUS15: U1001.20 (A15)
- new net NAME_BUS16: U1001.21 (A16)
- new net NAME_BUS17: U1001.22 (A17)
- new net NAME_BUS18: U1001.23 (A18)
- new net NAME_BUS19: U1001.24 (A19)
- new net NAME_BUS2: U1001.5 (A2)
- new net NAME_BUS20: U1001.25 (A20)
- new net NAME_BUS21: U1001.26 (A21)
- new net NAME_BUS22: U1001.27 (A22)
- new net NAME_BUS23: U1001.28 (A23)
- new net NAME_BUS24: U1001.29 (A24)
- new net NAME_BUS25: U1001.30 (A25)
- new net NAME_BUS26: U1001.31 (A26)
- new net NAME_BUS27: U1001.32 (A27)
- new net NAME_BUS28: U1001.33 (A28)
- new net NAME_BUS29: U1001.34 (A29)
- new net NAME_BUS3: U1001.7 (A3)
- new net NAME_BUS30: U1001.35 (A30)
- new net NAME_BUS31: U1001.36 (A31)
- new net NAME_BUS4: U1001.9 (A4)
- new net NAME_BUS5: U1001.10 (A5)
- new net NAME_BUS6: U1001.11 (A6)
- new net NAME_BUS7: U1001.12 (A7)
- new net NAME_BUS8: U1001.13 (A8)
- new net NAME_BUS9: U1001.14 (A9)
- new net NAME_PEV0: U3801.3 (P0), U907.8 (D1)
- new net NAME_PEV1: U3801.5 (P1), U907.10 (D2)
- new net NAME_PEV2: U3801.7 (P2), U907.12 (D3)
- new net NAME_PEV3: U3801.9 (P3), U907.14 (D4)
- new net OFFSET_BUS37: U906.71 (OFFS0)
- new net OFFSET_BUS38: U906.73 (OFFS1)
- new net OFFSET_BUS39: U906.74 (OFFS2)
- new net OFFSET_BUS40: U906.75 (OFFS3)
- new net OFFSET_BUS41: U906.76 (OFFS4)
- new net OFFSET_BUS42: U906.77 (OFFS5)
- new net OFFSET_BUS43: U906.78 (OFFS6)
- new net OFFSET_BUS44: U906.79 (OFFS7)
- new net OFFSET_BUS45: U906.80 (OFFS8)
- new net OFFSET_BUS46: U906.81 (OFFS9)
- new net OFFSET_BUS47: U906.82 (OFFS10)
- new net OFFSET_BUS48: U906.83 (OFFS11)
- new net OFFSET_BUS49: U906.84 (OFFS12)
- new net OFFSET_BUS50: U906.85 (OFFS13)
- new net OFFSET_BUS51: U906.86 (OFFS14)
- new net OFFSET_BUS52: U906.87 (OFFS15)
- new net OFFSET_BUS53: U906.88 (OFFS16)
- new net OFFSET_BUS54: U906.89 (OFFS17)
- new net OFFSET_BUS55: U906.90 (OFFS18)
- new net OFFSET_BUS56: U906.91 (OFFS19)
- new net OFFS_PEV0: U906.67 (PAR0), U907.16 (D5)
- new net OFFS_PEV1: U906.69 (PAR1), U907.18 (D6)
- new net OFFS_PEV2: U906.70 (PAR2), U907.20 (D7)
- new net Q.ADR.P0: GB161.1, U907.7 (Q0)
- new net Q.ADR.P1: GB158.1, U907.9 (Q1)
- new net Q.ADR.P2: GB157.1, U907.11 (Q2)
- new net Q.ADR.P3: GB155.1, U907.13 (Q3)
- new net Q.ADR.P4: GB154.1, U907.15 (Q4)
- new net Q.ADR.P5: GB153.1, U907.17 (Q5)
- new net Q.ADR.P6: GB147.1, U907.19 (Q6)
- new net Q.ADR.P7: GB146.1, U907.21 (Q7)
- new net Q.ADR.P8: GB145.1, U907.23 (Q8)
- new net Q4~: U1716.1 (D0), U3829.11 (CLK), U907.1 (CLK)
- no-connect marks 20 -> 18
Other:
- moved on the sheet: GB101, GB102, GB104, GB105, GB14, GB15, GB16, GB165, GB167, GB168, GB171, GB173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
