File: Schematics/Optimized/Mem32/pg_28.kicad_sch (KiCad schematic)
At the start: 20 parts, among them U2901 F20, U2902 F20, U2909 TAGAPAL, U2910 DRADPAL, U2911 PHITPAL, U2912 F04, U2913 SETPAL, U2914 F04, U2915 F51, U2916 F51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

Commit message: Integrate MEM32 condensations
Tested: passed run_udiag
Parts:
- removed U2912, U2914, U2921, U2922: F04, symbol r1000:F04
- removed U2913: SETPAL, symbol r1000:SETPAL
- removed U2915, U2916: F51, symbol r1000:F51
- removed U2917, U2918: F38, symbol r1000:F38
- removed U2919, U2920: F00, symbol r1000:F00
- added U1905, U1906: F374, symbol r1000:F374
- added U2003: XM28, symbol r1000:XM28
Connections:
- net AE_HIT~: now also U2003.30 (AEH)
- net AHIT~: now also U2003.10 (AHT)
- net AL_HIT~: now also U2003.31 (ALH)
- net BE_HIT~: now also U2003.32 (BEH)
- net BHIT~: now also U2003.14 (BHT)
- net BL_HIT~: now also U2003.33 (BLH)
- net B_AHIT~: now also U2003.12 (BAHT)
- net B_BHIT~: now also U2003.16 (BBHT)
- net B_SET2: now also U2003.19 (SET2)
- net B_SET3: now also U2003.21 (SET3)
- net CLK2X~: now also U1906.11 (CLK)
- net COMMAND0: now also U2003.26 (CMD0)
- net COMMAND1: now also U2003.27 (CMD1)
- net COMMAND2: now also U2003.28 (CMD2)
- net COMMAND3: now also U2003.29 (CMD3)
- net DRIVE_HIT: now also U2003.11 (DRH)
- net D_BUS_MODE0: now also U2003.22 (DBM0)
- net D_BUS_MODE1: now also U2003.23 (DBM1)
- net D_BUS_MODE2: now also U2003.24 (DBM2)
- net D_BUS_MODE3: now also U2003.25 (DBM3)
- net EXT_HIT: now also U2003.34 (EHIT)
- net H1: now also U2003.5 (H1)
- net HIGH_BOARD: now also U2003.13 (HIGH)
- net MCYC2_NEXT~: now also U2003.9 (MC2N)
- net MCYC2~: now also U2003.7 (MC2)
- net PD: now also U1905.1 (OE), U1906.1 (OE)
- net PHYS_SET0: now also U2003.15 (PSET0)
- net PHYS_SET1: now also U2003.17 (PSET1)
- net PHYS_SET2: now also U2003.18 (PSET2)
- net PHYS_SET3: now also U2003.20 (PSET3)
- net Q1~: now also U2003.3 (Q1)
- net TAGA12_Y: now also U1905.3 (D0)
- net TAGA13_Y: now also U1906.3 (D0)
- new net CLK2X: U1905.11 (CLK), U2003.1 (CLK)
- new net TAGA12: U1905.2 (Q0)
- new net TAGA13: U1906.2 (Q0)
- no-connect marks 10 -> 34
Other:
- moved on the sheet: U2901, U2902, U2909, U2910, U2911, U40, U41, U42, U43

Commit message: MEM32 improvements (also less F245 and F579 tri-state)
Parts:
- added U1902: F00, symbol r1000:F00
- added U1904: F04, symbol r1000:F04
- added U1905, U1906, U1907, U1908, U1909: F64, symbol r1000:F64
- added U1910, U1911, U1912, U1913, U1914: F37, symbol r1000:F37
Connections:
- net AHIT~: now also U1905.5 (C1), U1906.5 (C1), U1907.4 (C0)
- net BHIT~: now also U1904.1 (D0), U1907.6 (C2), U1908.6 (C2), U1909.6 (C2)
- net DRA2_EL_SEL: now also U2902.1 (D0); no longer U2902.5 (D3)
- net EXT_HIT: now also U1902.3 (Q), U1905.3 (A1), U1906.3 (A1), U1907.3 (A1), U1908.3 (A1), U1909.3 (A1)
- net HIGH_BOARD: now also U1905.6 (C2), U1906.6 (C2), U1907.5 (C1)
- net LOGQ_BE: now also U2902.2 (D1); no longer U2902.1 (D0)
- net NMATCHBE: now also U2902.4 (D2); no longer U2902.2 (D1)
- net OMATCHBE: now also U2902.5 (D3); no longer U2902.4 (D2)
- net PD: now also U1907.10 (B1), U1907.9 (B0), U1908.10 (B1), U1908.9 (B0), U1909.10 (B1), U1909.9 (B0)
- net TAGA12: now also U1905.19 (Q7); no longer U1905.2 (Q0)
- net TAGA12_Y: now also U1905.18 (D7); no longer U1905.3 (D0)
- new net: U1908.8 (Q), U1913.1 (D0)
- new net: U1905.8 (Q), U1910.1 (D0)
- new net: U1907.8 (Q), U1912.1 (D0)
- new net: U1906.8 (Q), U1911.1 (D0)
- new net: U1909.8 (Q), U1914.1 (D0)
- new net BSTOPA: U1904.2 (Q), U1905.10 (B1), U1906.10 (B1)
- new net BUZZ_OFF~: U1910.2 (D1), U1911.2 (D1), U1912.2 (D1), U1913.2 (D1), U1914.2 (D1)
- new net B_TVDRV~: U1905.1 (D0), U1906.1 (D0), U1908.12 (D2), U1909.1 (D0)
- new net B_VDRV~: U1906.12 (D2), U1907.12 (D2), U1909.12 (D2)
- new net B_XHITA~: U1902.1 (D0)
- new net B_XHITB~: U1902.2 (D1)
- new net D_DRVMEM~: U1905.13 (D3), U1906.11 (D1), U1907.1 (D0), U1908.13 (D3), U1909.11 (D1)
- new net D_DRVTAG~: U1906.13 (D3), U1907.13 (D3), U1909.13 (D3)
- new net TYP_AOE~: U1910.3 (Q)
- new net TYP_BOE~: U1913.3 (Q)
- new net VAL_AOE~: U1911.3 (Q)
- new net VAL_BOE~: U1914.3 (Q)
- new net VAL_POE~: U1912.3 (Q)
- no-connect marks 34 -> 52
Other:
- moved on the sheet: U1905, U1906, U2003, U2901, U2902, U2909, U2910, U2911, U40, U41, U42, U43

Commit message: Speedup: Condense multiplier, clocked parity comparison and more.
Other:
- moved on the sheet: U1902, U1904

Commit message: MEM32 condensation
Parts:
- removed U1905, U1906: F374, symbol r1000:F374
Connections:
- no-connect marks 52 -> 24
