File: Schematics/Optimized/Mem32/pg_30.kicad_sch (KiCad schematic)
At the start: 22 parts, among them U3101 RDRPAL, U3102 DRCPAL, U3103 F02, U3104 F02, U3105 F02, U3106 F02, U3107 F00, U3108 F00, U3109 F00, U3110 F00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

Commit message: MEM32 improvements
Parts:
- removed U3102: DRCPAL, symbol r1000:DRCPAL
- removed U3107, U44, U45: F00, symbol r1000:F00
- removed U3113: DLY_35, symbol r1000:DLY_35
- removed U3114: F175, symbol r1000:F175
- added U2201: XM30, symbol r1000:XM30
Connections:
- net RDRTBCLK is gone; now on net RDRTACLK: U3108.3 (Q)
- net AACAS~: now also U2201.4 (CASA)
- net AARAS~: now also U2201.2 (RAS)
- net AAWE~: now also U2201.9 (AWE)
- net AHIT~: now also U2201.16 (AHIT)
- net BACAS~: now also U2201.7 (CASB)
- net BHIT~: now also U2201.18 (BHIT)
- net CLK2X~: now also U2201.1 (CLK)
- net COL_ADR_OE~: now also U2201.17 (CAOE)
- net COMMAND0: now also U2201.3 (CMD0)
- net COMMAND1: now also U2201.5 (CMD1)
- net COMMAND2: now also U2201.6 (CMD2)
- net COMMAND3: now also U2201.8 (CMD3)
- net D_DIS_ADR: now also U2201.20 (DDA)
- net H1: now also U2201.10 (H1)
- net LATE_ABORT: now also U2201.19 (LAB)
- net MCYC2_NEXT~: now also U2201.12 (MCN)
- net MCYC2~: now also U2201.14 (MC)
- net NAMEQ~: now also U2201.11 (NMEQ)
- net ROW_ADR_OE~: now also U2201.15 (RAOE)
- net TAG_WRITE: now also U2201.13 (TAGW)
- no-connect marks 18 -> 7

Commit message: MEM32 improvements (also less F245 and F579 tri-state)
Parts:
- added U2004: F10, symbol r1000:F10
- added U2006: F20, symbol r1000:F20
- added U2007: F374, symbol r1000:F374
- added U2008, U2202: F02, symbol r1000:F02
- added U2203: BUSPAL, symbol r1000:BUSPAL
- added U2204: XBUF8, symbol r1000:XBUF8
- added U2205, U2206, U2207, U2208, U2209, U2210: F00, symbol r1000:F00
Connections:
- net COMMAND0: now also U2203.2 (I1)
- net COMMAND1: now also U2203.3 (I2)
- net COMMAND2: now also U2203.4 (I3)
- net COMMAND3: now also U2203.5 (I4)
- net H2: now also U2006.4 (D2)
- net LATE_ABORT: now also U2007.19 (Q7), U2008.2 (D1)
- net MCYC2_NEXT~: now also U2203.6 (I5)
- net PD: now also U2007.1 (OE), U2204.1 (INV), U2204.2 (OE)
- net SETA_SEL~: now also U2203.11 (I10)
- net SETB_SEL~: now also U2203.13 (I11)
- net TAGXEOE_EN: now also U2206.2 (D1), U2209.2 (D1)
- net TAGXLOE_EN: now also U2207.2 (D1), U2210.2 (D1)
- net TAGXOE_EN: now also U2205.2 (D1), U2208.2 (D1)
- new net ABORT~: U2008.3 (Q)
- new net B_EABT~: U2004.2 (D1)
- new net B_ELABT~: U2004.3 (D2), U2006.1 (D0)
- new net B_LABT~: U2006.2 (D1)
- new net DREG_OE: U2203.15 (D8), U2204.15 (I6)
- new net DREG_OE~: U2204.16 (Y6)
- new net D_BUS_MODE0: U2007.3 (D0), U2203.7 (I6)
- new net D_BUS_MODE1: U2203.8 (I7)
- new net D_BUS_MODE2: U2203.9 (I8)
- new net D_BUS_MODE3: U2203.10 (I9)
- new net D_EARLY_ABRT~: U2004.1 (D0)
- new net D_LATE_ABRT~: U2006.5 (D3)
- new net EABORT_Y: U2004.4 (Q), U2007.17 (D6)
- new net EARLY_ABORT: U2007.16 (Q6), U2008.1 (D0)
- new net EXT_SEL: U2204.10 (Y3)
- new net INHIBIT_VPAR: U2007.2 (Q0), U2202.1 (D0)
- new net INT_AOE: U2204.12 (Y4)
- new net INT_AOE~: U2203.19 (D4), U2204.11 (I4)
- new net INT_ASEL: U2204.8 (Y2)
- new net INT_BOE: U2204.14 (Y5)
- new net INT_BOE~: U2202.2 (D1), U2203.18 (D5), U2204.13 (I5)
- new net INT_BSEL: U2204.18 (Y7)
- new net INT_VPOE: U2202.3 (Q)
- new net LABORT_Y: U2006.6 (Q), U2007.18 (D7)
- new net MAR_P7_HD: U2007.12 (Q4)
- new net MAR_PAR7: U2007.13 (D4)
- new net Q4~: U2007.11 (CLK), U2203.1 (I0/CLK)
- new net RDR_SEL~: U2203.20 (D3), U2204.9 (I3)
- new net TAGAE_OE~: U2206.3 (Q)
- new net TAGAL_OE~: U2207.3 (Q)
- new net TAGA_DIR: U2204.4 (Y0)
- new net TAGA_DIR~: U2203.23 (D0), U2204.3 (I0)
- new net TAGA_OE: U2203.17 (D6), U2205.1 (D0), U2206.1 (D0), U2207.1 (D0)
- new net TAGA_OE~: U2205.3 (Q)
- new net TAGBE_OE~: U2209.3 (Q)
- new net TAGBL_OE~: U2210.3 (Q)
- new net TAGB_DIR: U2204.6 (Y1)
- new net TAGB_DIR~: U2203.22 (D1), U2204.5 (I1)
- new net TAGB_OE: U2203.16 (D7), U2208.1 (D0), U2209.1 (D0), U2210.1 (D0)
- new net TAGB_OE~: U2208.3 (Q)
- new net WDRA_SEL~: U2203.21 (D2), U2204.7 (I2)
- new net WDRB_SEL~: U2203.14 (D9), U2204.17 (I7)
- no-connect marks 7 -> 15
Other:
- moved on the sheet: U2201, U3101, U3103, U3104, U3105, U3106, U3108, U3109, U3110, U3111, U3112, U3115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

Commit message: MEM32 condensation
Parts:
- removed U2203: BUSPAL, symbol r1000:BUSPAL
- removed U2204: XBUF8, symbol r1000:XBUF8
- removed U3101: RDRPAL, symbol r1000:RDRPAL
- added U1703: XBUSPAL, symbol r1000:XBUSPAL
- added U2104: F374, symbol r1000:F374
Connections:
- net CKE2X: no longer U3108.1 (D0), U3109.1 (D0), U3110.1 (D0), U3111.1 (D0)
- net CLK2X: now also U2104.11 (CLK)
- net COMMAND0: now also U1703.3 (CMD0)
- net COMMAND1: now also U1703.5 (CMD1)
- net COMMAND2: now also U1703.6 (CMD2)
- net COMMAND3: now also U1703.8 (CMD3)
- net DREG_OE~: now also U1703.24 (DROEN)
- net D_BUS_MODE0: now also U1703.12 (DBMD0)
- net D_BUS_MODE1: now also U1703.13 (DBMD1)
- net D_BUS_MODE2: now also U1703.15 (DBMD2)
- net D_BUS_MODE3: now also U1703.16 (DBMD3)
- net D_DIS_ADR: now also U2201.22 (DDA); no longer U2201.20 (DDA)
- net EXT_SEL: now also U1703.25 (EXTSL)
- net INT_AOE: now also U1703.22 (INTAN)
- net INT_ASEL: now also U1703.19 (INTAS)
- net INT_BOE: now also U1703.23 (INTBN)
- net INT_BOE~: now also U1703.7 (INTB)
- net INT_BSEL: now also U1703.21 (INTBS)
- net LABORT_Y: now also U2104.3 (D0)
- net LATE_ABORT: now also U2201.20 (LAB); no longer U2201.19 (LAB)
- net MCYC2_NEXT~: now also U1703.10 (MC2N)
- net PD: now also U2104.1 (OE)
- net Q4~: now also U1703.1 (Q4)
- net RDR_CLKEN~: now also U2104.2 (Q0)
- net SETA_SEL~: now also U1703.18 (SETA)
- net SETB_SEL~: now also U2201.24 (SETB), U1703.20 (SETB)
- net TAGA_DIR: now also U1703.14 (TADIN)
- net TAGA_DIR~: now also U1703.2 (TADIR)
- net TAGA_OE: now also U1703.9 (TAOE)
- net TAGB_DIR: now also U1703.17 (TBDIN)
- net TAGB_DIR~: now also U1703.4 (TBDIR)
- net TAGB_OE: now also U1703.11 (TBOE)
- net TRDR_CLKEN~: now also U2201.19 (TRCE)
- net VARDR_CLKEN~: now also U2201.21 (VACE)
- net VBRDR_CLKEN~: now also U2201.23 (VBCE)
- net VPRDR_CLKEN~: now also U2201.25 (VPCE)
- net INHIBIT_VPAR: no longer names the net of U2007.2 (Q0), U2202.1 (D0)
- new net PU: U3108.1 (D0), U3109.1 (D0), U3110.1 (D0), U3111.1 (D0)
- no-connect marks 15 -> 25
Other:
- note added: "lo=15…115ns"
- note added: "lo=15…55ns"
- moved on the sheet: U2004, U2006, U2007, U2008, U2202, U2205, U2206, U2207, U2208, U2209, U2210, U3103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

Commit message: MEM32 cache condensation
Parts:
- removed U2205, U2206, U2207, U2208, U2209, U2210, U3108, U3109, U3110, U3111: F00, symbol r1000:F00
- removed U3103, U3104, U3105, U3106: F02, symbol r1000:F02
- removed U3112: TSCPAL, symbol r1000:TSCPAL
- added U1001: F00, symbol r1000:F00
- added U1002, U1003, U1004, U1005: F32, symbol r1000:F32
- added U1904: F04, symbol r1000:F04
- added U1905, U1906, U1907, U1908, U1909: F64, symbol r1000:F64
- added U1910, U1911, U1912, U1913, U1914: F37, symbol r1000:F37
- added U2003: XM28, symbol r1000:XM28
- added U2909: TAGAPAL, symbol r1000:TAGAPAL
- added U2910: DRADPAL, symbol r1000:DRADPAL
- added U2911: PHITPAL, symbol r1000:PHITPAL
Connections:
- net AHIT~: now also U1905.5 (C1), U1906.5 (C1), U1907.4 (C0), U2003.10 (AHT)
- net BHIT~: now also U1904.1 (D0), U1907.6 (C2), U1908.6 (C2), U1909.6 (C2), U2003.14 (BHT)
- net CLK2X: now also U2003.1 (CLK)
- net CLK2X~: now also U2909.1 (I0/CLK), U2910.1 (I0/CLK)
- net COMMAND0: now also U2003.28 (CMD0), U2909.2 (I1), U2910.2 (I1)
- net COMMAND1: now also U2003.30 (CMD1), U2909.3 (I2), U2910.3 (I2)
- net COMMAND2: now also U2003.31 (CMD2), U2909.4 (I3), U2910.4 (I3)
- net COMMAND3: now also U2003.33 (CMD3), U2909.5 (I4)
- net D_BUS_MODE0: now also U2003.22 (DBM0), U2911.7 (I6)
- net D_BUS_MODE1: now also U2003.23 (DBM1), U2911.8 (I7)
- net D_BUS_MODE2: now also U2003.25 (DBM2), U2911.9 (I8)
- net D_BUS_MODE3: now also U2003.26 (DBM3), U2909.21 (D2), U2911.11 (I9)
- net D_DIS_ADR: now also U2910.5 (I4)
- net H1: now also U2003.5 (H1), U2909.6 (I5), U2910.6 (I5), U2911.6 (I5)
- net LATE_ABORT: now also U2003.44 (LABRT), U2909.13 (I11)
- net MCYC2_NEXT~: now also U2003.9 (MC2N), U2909.7 (I6)
- net MCYC2~: now also U2003.7 (MC2), U2909.8 (I7), U2910.7 (I6)
- net PD: now also U1907.10 (B1), U1907.9 (B0), U1908.10 (B1), U1908.9 (B0), U1909.10 (B1), U1909.9 (B0)
- net PHYS_SET3: now also U2003.20 (PSET3), U2909.10 (I9), U2911.4 (I3)
- net RDRTACLK: now also U1002.3 (Q)
- net RDRVACLK: now also U1003.3 (Q)
- net RDRVBCLK: now also U1004.3 (Q)
- net RDRVPCLK: now also U1005.3 (Q)
- net RDR_CLKEN~: now also U1002.2 (D1), U1003.2 (D1), U1004.2 (D1), U1005.2 (D1)
- net SETA_SEL~: now also U2911.16 (D2)
- net SETB_SEL~: now also U2911.15 (D3)
- net TAGA_CE: now also U2003.38 (TGACE)
- net TAGB_CE: now also U3119.2 (D1), U2003.40 (TGBCE); no longer U3119.1 (D0)
- net TAGXEOE_EN: now also U2003.24 (TXEOE)
- net TAGXE_WE: now also U2003.34 (TXEWE)
- net TAGXLOE_EN: now also U2003.27 (TXLOE)
- net TAGXL_WE: now also U2003.36 (TXLWE)
- net TAGXX_WE: now also U2003.32 (TXXWE)
- net TRDR_CLKEN~: now also U1002.1 (D0)
- net TS_CE_EN: now also U3119.1 (D0); no longer U3119.2 (D1)
- net VARDR_CLKEN~: now also U1003.1 (D0)
- net VBRDR_CLKEN~: now also U1004.1 (D0)
- net VPRDR_CLKEN~: now also U1005.1 (D0)
- net TSC14: now reaches U3115.1 (A1)
- net TSC14: now also U2003.42 (TSC14)
- net TAGA_DIR~: no longer names the net of U1703.2 (TADIR)
- net TAGB_DIR~: no longer names the net of U1703.4 (TBDIR)
- new net: U1906.8 (Q), U1911.1 (D0)
- new net: U1909.8 (Q), U1914.1 (D0)
- new net: U1907.8 (Q), U1912.1 (D0)
- new net: U1908.8 (Q), U1913.1 (D0)
- new net: U1905.8 (Q), U1910.1 (D0)
- new net AE_HIT~: U2003.35 (AEH), U2910.17 (D6)
- new net AL_HIT~: U2003.37 (ALH), U2910.16 (D7)
- new net BE_HIT~: U2003.39 (BEH), U2910.15 (D8)
- new net BL_HIT~: U2003.41 (BLH), U2910.14 (D9)
- new net BSTOPA: U1904.2 (Q), U1905.10 (B1), U1906.10 (B1)
- new net BUZZ_OFF~: U1910.2 (D1), U1911.2 (D1), U1912.2 (D1), U1913.2 (D1), U1914.2 (D1)
- new net B_AHIT~: U2003.12 (BAHT)
- new net B_BHIT~: U2003.16 (BBHT)
- new net B_SET2: U2003.19 (SET2)
- new net B_SET3: U2003.21 (SET3)
- new net B_TVDRV~: U1905.1 (D0), U1906.1 (D0), U1908.12 (D2), U1909.1 (D0)
- new net B_VDRV~: U1906.12 (D2), U1907.12 (D2), U1909.12 (D2)
- new net B_XHITA~: U1001.1 (D0)
- new net B_XHITB~: U1001.2 (D1)
- new net CHECK_TSEPAR: U2909.17 (D6)
- new net DRA2_EL_SEL: U2910.23 (D0)
- new net DRA_A1: U2910.21 (D2)
- new net DRA_A2LP: U2910.19 (D4)
- new net DRB_A1: U2910.20 (D3)
- new net DRB_A2LP: U2910.18 (D5)
- new net DRIVE_HIT: U2003.11 (DRH)
- new net D_DRVMEM~: U1905.13 (D3), U1906.11 (D1), U1907.1 (D0), U1908.13 (D3), U1909.11 (D1)
- new net D_DRVTAG~: U1906.13 (D3), U1907.13 (D3), U1909.13 (D3)
- new net D_FORCE_HIT~: U2911.13 (D5)
- new net EXT_HIT: U1001.3 (Q), U1905.3 (A1), U1906.3 (A1), U1907.3 (A1), U1908.3 (A1), U1909.3 (A1), U2003.43 (EHIT)
- new net HIGH_BOARD: U1905.6 (C2), U1906.6 (C2), U1907.5 (C1), U2003.13 (HIGH), U2911.5 (I4)
- new net LAR_2: U2910.9 (I8)
- new net LAR_3: U2910.10 (I9)
- new net LRU_UPDATE: U2909.16 (D7)
- new net PHIT_AE~: U2911.19 (O0)
- new net PHIT_AL~: U2911.12 (O1)
- new net PHIT_BE~: U2911.18 (D0)
- new net PHIT_BL~: U2911.17 (D1)
- new net PHYS_HIT26~: U2910.8 (I7), U2911.14 (D4)
- new net PHYS_SET0: U2003.15 (PSET0), U2911.1 (I0)
- new net PHYS_SET1: U2003.17 (PSET1), U2911.2 (I1)
- new net PHYS_SET2: U2003.18 (PSET2), U2909.9 (I8), U2911.3 (I2)
- new net Q1~: U2003.3 (Q1)
- new net TAGA12_Y: U2909.19 (D4)
- new net TAGA13_Y: U2909.18 (D5)
- new net TRACE_DRA1: U2910.11 (I10)
- new net TRACE_DRA2: U2910.13 (I11)
- new net TS_TRACE_EN: U2909.11 (I10)
- new net TS_TRADR12E: U2909.23 (D0)
- new net TS_TRADR12L: U2909.22 (D1)
- new net TS_TRADR13E: U2909.15 (D8)
- new net TS_TRADR13L: U2909.14 (D9)
- new net TYP_AOE~: U1910.3 (Q)
- new net TYP_BOE~: U1913.3 (Q)
- new net VAL_AOE~: U1911.3 (Q)
- new net VAL_BOE~: U1914.3 (Q)
- new net VAL_POE~: U1912.3 (Q)
- no-connect marks 25 -> 51
Other:
- moved on the sheet: U2004, U2006, U2007, U2008, U2104, U2201, U2202, U3115, U3116, U3119, U3120, U3124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

Commit message: Typ/Val/Mem32 improvements
Parts:
- removed U1001: F00, symbol r1000:F00
- removed U1904: F04, symbol r1000:F04
- removed U1905, U1906, U1907, U1908, U1909: F64, symbol r1000:F64
- removed U1910, U1911, U1912, U1913, U1914: F37, symbol r1000:F37
- removed U2004: F10, symbol r1000:F10
- removed U2006: F20, symbol r1000:F20
- removed U2008: F02, symbol r1000:F02
- removed U2104: F374, symbol r1000:F374
- removed U2910: DRADPAL, symbol r1000:DRADPAL
- removed U2911: PHITPAL, symbol r1000:PHITPAL
- added U1008: XMBUSCTL, symbol r1000:XMBUSCTL
Connections:
- net ABORT~: now also U2003.54 (ABORT)
- net AHIT~: now also U1008.15 (AHIT)
- net BHIT~: now also U1008.16 (BHIT)
- net B_EABT~: now also U2003.47 (EABT)
- net B_ELABT~: now also U2003.49 (ELABT)
- net B_LABT~: now also U2003.51 (LABT)
- net B_TVDRV~: now also U1008.9 (TVDRV)
- net B_VDRV~: now also U1008.11 (VDRV)
- net B_XHITA~: now also U1008.13 (XHITA)
- net B_XHITB~: now also U1008.14 (XHITB)
- net DRA2_EL_SEL: now also U2003.66 (DA2SL)
- net DRA_A1: now also U2003.61 (DAA1D)
- net DRA_A2LP: now also U2003.64 (DAA2D)
- net DRB_A1: now also U2003.63 (DBA1D)
- net DRB_A2LP: now also U2003.65 (DBA2D)
- net D_DIS_ADR: now also U2003.55 (DDISA)
- net D_DRVMEM~: now also U1008.3 (DDRVMEM)
- net D_DRVTAG~: now also U1008.5 (DDRVTAG)
- net D_EARLY_ABRT~: now also U2003.45 (DEABT)
- net D_FORCE_HIT~: now also U2003.50 (DFHIT)
- net D_LATE_ABRT~: now also U2003.53 (DLABT)
- net EARLY_ABORT: now also U2003.56 (EABRT); no longer U2007.16 (Q6)
- net EXT_HIT: now also U1008.12 (EXTHIT)
- net HIGH_BOARD: now also U1008.7 (HIBOARD)
- net LAR_2: now also U2003.60 (LAR2)
- net LAR_3: now also U2003.62 (LAR3)
- net LATE_ABORT: now also U2003.59 (LABRT); no longer U2003.44 (LABRT), U2007.19 (Q7)
- net PHIT_AE~: now also U2003.2 (PHAE)
- net PHIT_AL~: now also U2003.4 (PHAL)
- net PHIT_BE~: now also U2003.6 (PHBE)
- net PHIT_BL~: now also U2003.8 (PHBL)
- net PHYS_HIT26~: now also U2003.48 (PHT26)
- net RDR_CLKEN~: now also U2003.52 (RCLKE)
- net SETA_SEL~: now also U2003.44 (SETAS)
- net SETB_SEL~: now also U2003.46 (SETBS)
- net TRACE_DRA1: now also U2003.57 (TRDR1)
- net TRACE_DRA2: now also U2003.58 (TRDR2)
- net TYP_AOE~: now also U1008.2 (TYPAOE)
- net TYP_BOE~: now also U1008.6 (TYPBOE)
- net VAL_AOE~: now also U1008.4 (VALAOE)
- net VAL_BOE~: now also U1008.8 (VALBOE)
- net VAL_POE~: now also U1008.10 (VALPOE)
- net EABORT_Y: no longer names the net of U2007.17 (D6)
- net LABORT_Y: no longer names the net of U2007.18 (D7)
- new net DIAG_BUZZ_OFF: U1008.1 (DBUZZOF)
- no-connect marks 51 -> 18
Other:
- moved on the sheet: U1002, U1003, U1004, U1005, U1703, U2007, U2201, U2202, U2909, U3115, U3116, U3119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

Commit message: XCLKSTP, XIOP XSUDEC
Connections:
- net PHYS_HIT26~: no longer names the net of U2003.48 (PHT26)
- no-connect marks 18 -> 19
Changed lines of the file:
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@@
   (no_connect (at 515.62 185.42))
   (no_connect (at 106.68 144.78))
+  (no_connect (at 106.68 236.22))
   (no_connect (at 482.6 254))
   (no_connect (at 347.98 337.82))
@@
     (stroke (width 0) (type default))
   )
-  (wire (pts (xy 106.68 236.22) (xy 137.16 236.22))
-    (stroke (width 0) (type default))
-  )
   (wire (pts (xy 58.42 160.02) (xy 63.5 160.02))
     (stroke (width 0) (type default))
@@
     (effects (font (size 2.54 2.54)) (justify left bottom))
   )
-  (label "PHYS_HIT26~" (at 111.76 236.22 0) (fields_autoplaced)
-    (effects (font (size 2.54 2.54)) (justify left bottom))
-  )
