File: Schematics/Hw/Ioc/pg_18.kicad_sch (KiCad schematic)
At the start: 12 parts, among them U1901 PA110, U1902 F163, U1903 F174, U1904 F175, U1905 F04, U1906 8641, U1907 8641, U1908 8641, U1909 8641, U1910 F374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

Commit message: Polish
Other:
- note added: "0xFFFFFC00"
Changed lines of the file:
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@@
     (stroke (width 0) (type default))
+  )
+  (text "0xFFFFFC00" (at 119.38 147.32 0)
+    (effects (font (size 2.54 2.54)) (justify left bottom))
   )
   (label "IO.EN" (at 104.14 40.64 0) (fields_autoplaced)
