File: Schematics/Optimized/Typ/pg_26.kicad_sch (KiCad schematic)
At the start: 5 parts, among them U1301 XPRIVCMP, U2812 F64, U2817 F02, U2818 F08, U2819 F64

Commit message: Optimization of TYP & VAL
Tested: boot_env (until PRETTY_PRINTER assert)
Tested: passed run_udiag
Other:
- moved on the sheet: U1301, U2812, U2817, U2818, U2819

Commit message: Condensation of SEQ, TYP & VAL conditions
Parts:
- added GB106, GB166, GB172, GB176, GB178, GB181, GB182, GB183, GB188, GB191, GB192, GB196, GB202, GB54, GB57, GB58, GB61, GB62, GB63: GB, symbol r1000:GB
- added U1111: XTCOND, symbol r1000:XTCOND
- added U2901, U2902, U2917, U2918: F04, symbol r1000:F04
- added U2903, U2904, U2905, U2906, U2915: F02, symbol r1000:F02
- added U2907, U2910, U2911, U2912: F10, symbol r1000:F10
- added U2908: F138, symbol r1000:F138
- added U2909, U2916, U2919, U2921: F00, symbol r1000:F00
- added U2913, U2914: F51, symbol r1000:F51
- added U2920: F194, symbol r1000:F194
- added U2922: F174, symbol r1000:F174
Connections:
- net B_BIN_MATCH is gone; now on net A_OP_PASS~: U1301.135 (AOP)
- net DERIVE_PRIV is gone; now on net B_OP_PASS~: U1301.138 (BOP)
- net A_OP_PASS~: now also U1111.46 (C2F), U2913.2 (A2), U2914.4 (B1); no longer U1301.134 (AOP)
- net BIN_EQ_PASS~: now also U1111.48 (C2H), U2911.3 (D2)
- net BIN_OP_PASS~: now also U1301.141 (IOP), U1111.49 (C3A), U2910.3 (D2); no longer U1301.137 (IOP)
- net B_OP_PASS~: now also U1111.47 (C2G), U2913.4 (B1), U2914.2 (A2); no longer U1301.136 (BOP)
- net CLASS_CHECK.EN: now also U1301.152 (CLCE), U2912.3 (D2)
- net CLASS_EVENT: now also U1301.153 (CLEV), U2912.2 (D1)
- net MICROS_EN: now also U2902.2 (Q), U2910.1 (D0), U2911.1 (D0), U2912.1 (D0), U2921.1 (D0)
- net PD: now also U2908.5 (D2)
- net PRIV_NAMES_EQ: now also U1111.50 (C3B)
- net PRIV_PATH_EQ~: now also U1111.51 (C3C)
- net PRIV_STRUCT: now also U1111.52 (C3D)
- net SELECT_A_OP: now also U2919.3 (Q)
- net SELECT_BIN_EQ: now also U2911.2 (D1), U2917.2 (Q)
- net SELECT_BIN_OP: now also U2910.2 (D1), U2918.2 (Q)
- net SELECT_B_OP: now also U2916.3 (Q)
- net SYSTEM_MICRO: now also U1301.154 (SYSU), U2921.2 (D1)
- net A_BIN_MATCH renamed C_LIT~1
- net A_OP_MATCH renamed OF~.SCLK
- net B_OP_MATCH renamed C_LIT~0
- new net: U2904.3 (Q), U2913.5 (B2)
- new net: U2903.3 (Q), U2913.1 (A1)
- new net: U2913.7 (Q), U2922.11 (D3)
- new net: U2910.4 (Q), U2922.3 (D0)
- new net: U2921.3 (Q), U2922.14 (D5)
- new net: U2914.7 (Q), U2922.13 (D4)
- new net: U2911.4 (Q), U2922.4 (D1)
- new net: U2912.4 (Q), U2922.6 (D2)
- new net: U2915.3 (Q), U2920.10 (S1), U2920.9 (S0)
- new net: U2906.3 (Q), U2914.5 (B2)
- new net: U2909.3 (Q), U2915.2 (D1)
- new net: U2905.3 (Q), U2914.1 (A1)
- new net ALU.D0: U1111.31 (C1C)
- new net ALU.ZERO0: U1111.30 (ALUZ0)
- new net ALU.ZERO1: U1111.32 (ALUZ1)
- new net ALU.ZERO2: U1111.33 (ALUZ2)
- new net ALU.ZERO3: U1111.35 (ALUZ3)
- new net ALU.ZERO4: U1111.36 (ALUZ4)
- new net ALU.ZERO5: U1111.38 (ALUZ5)
- new net ALU.ZERO6: U1111.39 (ALUZ6)
- new net ALU.ZERO7: U1111.41 (ALUZ7)
- new net ALU_32_CO: U1111.23 (C0H)
- new net ALU_CO: U1111.26 (C1A)
- new net A_BUF0: U1111.34 (ABIT0)
- new net A_TOS_1_OP~: U2903.1 (D0), U2908.12 (Y3_), U2919.2 (D1)
- new net A_TOS_OP~: U2906.1 (D0), U2908.13 (Y2_), U2919.1 (D0)
- new net BBIT0: U1111.54 (BBIT0), U1301.155 (BBIT0)
- new net BBIT21: U1111.55 (BBIT1), U1301.156 (BBIT1)
- new net BBIT32: U1111.56 (BBIT2), U1301.157 (BBIT2)
- new net BBIT33: U1111.57 (BBIT3), U1301.158 (BBIT3)
- new net BBIT34: U1111.58 (BBIT4), U1301.159 (BBIT4)
- new net BBIT35: U1111.59 (BBIT5), U1301.160 (BBIT5)
- new net BBIT36: U1111.60 (BBIT6), U1301.161 (BBIT6)
- new net B_BUF61: U1301.162 (BBUF0)
- new net B_BUF62: U1301.163 (BBUF1)
- new net B_BUF63: U1301.164 (BBUF2)
- new net B_TOS_1_OP~: U2904.1 (D0), U2908.10 (Y5_), U2916.2 (D1)
- new net B_TOS_OP~: U2905.1 (D0), U2908.11 (Y4_), U2916.1 (D0)
- new net CLASS_ABLIT~: U1301.147 (UCOD3)
- new net CLASS_ABL_EQ: U1111.45 (C2E), U1301.151 (ABLE)
- new net CLASS_A_EQ_B~: U1111.44 (C2D), U1301.149 (AEQB)
- new net CLASS_A_EQ_L~: U1111.42 (C2B), U1301.146 (AEQL)
- new net CLASS_A_TO_B~: U1301.144 (UCOD1)
- new net CLASS_A_TO_L~: U1301.142 (UCOD0)
- new net CLASS_B_EQ_L~: U1111.43 (C2C), U1301.150 (BEQL)
- new net CLASS_B_TO_L~: U1301.145 (UCOD2)
- new net CLASS_SYS_B~: U1301.148 (UCOD4)
- new net COND~.SCLK: U1111.17 (SCLK)
- new net C_LIT~2: U1301.134 (CLIT2)
- new net C_LIT~3: U1301.136 (CLIT3)
- new net C_LIT~4: U1301.137 (CLIT4)
- new net C_LIT~5: U1301.139 (CLIT5)
- new net C_LIT~6: U1301.140 (CLIT6)
- new net DIAG_MODE: U2915.1 (D0)
- new net IS_BINARY: U1111.20 (ISBIN)
- new net LAST_TYP~: U1111.13 (LVCND)
- new net LOOP_CNT0: U1111.15 (LOOP0)
- new net LOOP_CNT1: U1111.16 (LOOP1)
- new net LOOP_CNT2: U1111.18 (LOOP2)
- new net LOOP_CNT3: U1111.19 (LOOP3)
- new net LOOP_CNT4: U1111.21 (LOOP4)
- new net LOOP_CNT5: U1111.22 (LOOP5)
- new net LOOP_CNT6: U1111.24 (LOOP6)
- new net LOOP_CNT7: U1111.25 (LOOP7)
- new net LOOP_CNT8: U1111.27 (LOOP8)
- new net LOOP_CNT9: U1111.28 (LOOP9)
- new net MICROS_EN~: U2901.2 (Q), U2902.1 (D0), U2903.2 (D1), U2904.2 (D1), U2905.2 (D1), U2906.2 (D1), U2908.4 (D1)
- new net OF_KIND_MATCH: U1111.40 (C2A), U1301.143 (OKM)
- new net OVR.EN~: U1111.29 (OVREN)
- new net PASS_PRIVACY~: U1111.53 (C3E), U2908.6 (D0), U2920.15 (Q0)
- new net PRIV_NO_OP~: U2907.4 (Q), U2909.1 (D0)
- new net Q3~: U2922.9 (CLK)
- new net Q4~: U2920.11 (CLK)
- new net SELECT_BIN_EQ~: U2908.15 (Y0_), U2917.1 (D0)
- new net SELECT_BIN_OP~: U2908.14 (Y1_), U2918.1 (D0)
- new net SET_PASS_PRV~: U2920.3 (D0)
- new net STATE_CLK.EN: U2909.2 (D1)
- new net SUB_ELSE_ADD~: U1111.37 (SELA)
- new net T.BIN_EQ.UE~: GB62.1, U2922.5 (Q1)
- new net T.BIN_OP.UE~: GB61.1, U2922.2 (Q0)
- new net T.CHK_SYS.UE~: GB54.1, U2922.15 (Q5)
- new net T.CLASS.UE~: GB63.1, U2922.7 (Q2)
- new net T.COND.SEL0: GB166.1, U1111.1 (SEL0)
- new net T.COND.SEL1: GB172.1, U1111.3 (SEL1)
- new net T.COND.SEL2: GB176.1, U1111.5 (SEL2)
- new net T.COND.SEL3: GB178.1, U1111.7 (SEL3)
- new net T.COND.SEL4: GB181.1, U1111.9 (SEL4)
- new net T.COND.SEL5: GB182.1, U1111.11 (SEL5)
- new net T.COND.SEL6: GB183.1, U1111.12 (SEL6)
- new net T.COND.TYPE0: GB188.1, U1111.2 (VCOND0)
- new net T.COND.TYPE1: GB191.1, U1111.4 (VCOND1)
- new net T.COND.TYPE2: GB192.1, U1111.6 (VCOND2)
- new net T.COND.TYPE3: GB196.1, U1111.8 (VCOND3)
- new net T.COND.TYPE4: GB202.1, U1111.10 (VCOND4)
- new net T.MICROS_EN: GB106.1, U2901.1 (D0)
- new net T.TOS1_OP.UE~: GB57.1, U2922.10 (Q3)
- new net T.TOS_OP.UE~: GB58.1, U2922.12 (Q4)
- new net UIR.PRIV_CHEK0: U2907.3 (D2), U2908.3 (S0)
- new net UIR.PRIV_CHEK1: U2907.2 (D1), U2908.2 (S1)
- new net UIR.PRIV_CHEK2: U2907.1 (D0), U2908.1 (S2)
- no-connect marks 1 -> 18
Other:
- note added: "CLEAR_PASS_PRIVACY~"
- note added: "COMBO CONDITION ENCODING = 1011XXX COMBO CONDITION XXX = LOGICAL NAND OF COMBINATION 0000XXX (VAL) AND CONDITION 0011XXX (TYP)"
- note added: "NO_OP~"
- note added: "TYPE BOARD CONDITION ENCODINGS ------------------------------ ENCODING TIMING NAME COMMENT -------- ------ ---- ------- 0011 000 LATE TYP_ALU_ZERO 0011 001 LATE TYP_ALU_NONEZERO 0011 010 LATE TYP_ALU_A_GT_OR_GE_B 0011 011 SPARE 0011 100 EARLY TYP_LOOP_COUNTER_ZERO 0011 101 SPARE 0011 110 LATE TYP_ALU_ZERO COMBO WITH VAL_ALU_NONZERO 0011 111 LATE TYP_ALU_32_CO ALU 32 BIT CARRY OUT 0100 000 LATE TY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"
- moved on the sheet: U2812, U2817, U2818, U2819

Commit message: Typ/Val/Mem32 improvements
Parts:
- removed U2812, U2819: F64, symbol r1000:F64
- removed U2817, U2903, U2904, U2905, U2906, U2915: F02, symbol r1000:F02
- removed U2818: F08, symbol r1000:F08
- removed U2901, U2902, U2917, U2918: F04, symbol r1000:F04
- removed U2907, U2910, U2911, U2912: F10, symbol r1000:F10
- removed U2908: F138, symbol r1000:F138
- removed U2909, U2916, U2919, U2921: F00, symbol r1000:F00
- removed U2913, U2914: F51, symbol r1000:F51
- removed U2920: F194, symbol r1000:F194
- removed U2922: F174, symbol r1000:F174
- added U78: XREG16, symbol r1000:XREG16
Connections:
- net BIN_EQ_PASS~ is gone; now on net BIN_OP_PASS~: U1111.48 (C3A)
- net CLASS_CHECK.EN is gone; now on net UIR.PRIV_CHEK0: U1301.152 (UPVC0)
- net CLASS_EVENT is gone; now on net CLASS_ABL_EQ: U1301.153 (ABLE)
- net PRIV_STRUCT is gone; now on net BBIT0: U1111.52 (BBIT0)
- net SYSTEM_MICRO is gone; now on net UIR.PRIV_CHEK1: U1301.154 (UPVC1)
- net BBIT0: now also U1301.158 (BBIT0); no longer U1111.54 (BBIT0), U1301.155 (BBIT0)
- net BBIT21: now also U1111.53 (BBIT1), U1301.159 (BBIT1); no longer U1111.55 (BBIT1), U1301.156 (BBIT1)
- net BBIT32: now also U1111.54 (BBIT2), U1301.161 (BBIT2); no longer U1111.56 (BBIT2), U1301.157 (BBIT2)
- net BBIT33: now also U1111.55 (BBIT3), U1301.162 (BBIT3); no longer U1111.57 (BBIT3), U1301.158 (BBIT3)
- net BBIT34: now also U1111.56 (BBIT4), U1301.164 (BBIT4); no longer U1111.58 (BBIT4), U1301.159 (BBIT4)
- net BBIT35: now also U1111.57 (BBIT5), U1301.165 (BBIT5); no longer U1111.59 (BBIT5), U1301.160 (BBIT5)
- net BBIT36: now also U1111.58 (BBIT6), U1301.167 (BBIT6); no longer U1111.60 (BBIT6), U1301.161 (BBIT6)
- net BIN_OP_PASS~: no longer U1111.49 (C3A)
- net B_BUF61: now also U1301.169 (BBUF0); no longer U1301.162 (BBUF0)
- net B_BUF62: now also U1301.170 (BBUF1); no longer U1301.163 (BBUF1)
- net B_BUF63: now also U1301.172 (BBUF2); no longer U1301.164 (BBUF2)
- net CLASS_ABL_EQ: no longer U1301.151 (ABLE)
- net CLASS_B_EQ_L~: now also U1301.151 (BEQL); no longer U1301.150 (BEQL)
- net DIAG_MODE: now also U1301.166 (DMODE)
- net PASS_PRIVACY~: now also U1111.51 (C3E), U1301.156 (PPRIV); no longer U1111.53 (C3E)
- net PD: now also U78.10 (D2), U78.8 (D1)
- net PRIV_NAMES_EQ: now also U1111.49 (C3B); no longer U1111.50 (C3B)
- net PRIV_PATH_EQ~: now also U1111.50 (C3C); no longer U1111.51 (C3C)
- net Q4~: now also U1301.150 (Q4), U78.1 (CLK)
- net SET_PASS_PRV~: now also U1301.160 (SPPRV)
- net STATE_CLK.EN: now also U1301.163 (SCKEN)
- net T.BIN_EQ.UE~: now also U1301.174 (UE1), U78.26 (D10)
- net T.BIN_OP.UE~: now also U1301.173 (UE0), U78.28 (D11)
- net T.CHK_SYS.UE~: now also U1301.178 (UE5), U78.36 (D15)
- net T.CLASS.UE~: now also U1301.175 (UE2), U78.34 (D14)
- net T.COND.TYPE0: now also U78.16 (D5)
- net T.COND.TYPE1: now also U78.18 (D6)
- net T.COND.TYPE2: now also U78.20 (D7)
- net T.COND.TYPE3: now also U78.22 (D8)
- net T.COND.TYPE4: now also U78.24 (D9)
- net T.MICROS_EN: now also U1301.157 (UEN)
- net T.TOS1_OP.UE~: now also U1301.176 (UE3), U78.32 (D13)
- net T.TOS_OP.UE~: now also U1301.177 (UE4), U78.30 (D12)
- net T.TYPE0_STOP~: now also U1301.168 (T0STP)
- net T.TYPE1_STOP~: now also U1301.171 (T1STP)
- net UIR.PRIV_CHEK2: now also U1301.155 (UPVC2)
- new net DIAG.D0: U78.7 (Q0)
- new net DIAG.D1: U78.9 (Q1)
- new net DIAG.D10: U78.27 (Q10)
- new net DIAG.D11: U78.29 (Q11)
- new net DIAG.D12: U78.31 (Q12)
- new net DIAG.D13: U78.33 (Q13)
- new net DIAG.D14: U78.35 (Q14)
- new net DIAG.D15: U78.37 (Q15)
- new net DIAG.D2: U78.11 (Q2)
- new net DIAG.D3: U78.13 (Q3)
- new net DIAG.D4: U78.15 (Q4)
- new net DIAG.D5: U78.17 (Q5)
- new net DIAG.D6: U78.19 (Q6)
- new net DIAG.D7: U78.21 (Q7)
- new net DIAG.D8: U78.23 (Q8)
- new net DIAG.D9: U78.25 (Q9)
- new net PERR_SCAN_OUT: U78.14 (D4)
- new net SCAN_CONTROL~: U78.3 (OE)
- no-connect marks 18 -> 4
Other:
- note removed: "(LIMITED_SCALAR_OP_PASS~)"
- note removed: "CLEAR_PASS_PRIVACY~"
- note removed: "NO_OP~"
- moved on the sheet: GB106, GB166, GB172, GB176, GB178, GB181, GB182, GB183, GB188, GB191, GB192, GB196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

Commit message: Update to kicad9
Parts:
- renumbered U78 to U601
